File: step-up_converter/step-up_converter.sch (KiCad schematic (older format))
At the start: 9 parts, among them U1 LM2731YMF

Commit message: Schematic update
Parts:
- removed D1: MBR0520LT, Diode_SMD:D_SOD-123, symbol MBR0520LT
- removed L1: 10u, symbol INDUCTOR
- removed U1: LM2731YMF, SOT-23-5, symbol LM2731YMF
- added D1: MBR0520, Diode_SMD:D_SOD-123, symbol Diode:MBR0520
- added L1: 10u, symbol pspice:INDUCTOR
- added P1: PWR_IN, symbol power_sources:PWR_IN
- added U1: LM2731YMF, Package_TO_SOT_SMD:SOT-23-5, symbol Regulator_Switching:LM2731YMF
- C1, C3: symbol C -> Device:C
- C2: value 220p -> 150p; symbol C -> Device:C
- R1, R2, R3: symbol R -> Device:R
Connections:
- net 0: now also P1.2 (GND), U1.2 (GND)
- net INPUT_18V: now also D1.1 (K)
- net VCC: now also L1.1, P1.1 (VCC), U1.4 (EN), U1.5 (VIN)
- net at C2.2, R1.1, R2.2: now also U1.3 (FB)
- new net: D1.2 (A), L1.2, U1.1 (SW)
Other:
- note added: ".include power.cir\n.tran 10us 200us uic"
